File: Load Cell/corbin.sch (KiCad schematic (older format))
At the start: 4 parts, among them J11 Conn_01x04, J16 Conn_01x06

Commit message: 2-17-22
Connections:
- net A+: now also J16.4 (Pin_4); no longer J16.3 (Pin_3)
- net A-: now also J16.3 (Pin_3); no longer J16.4 (Pin_4)
- net GND: now also J11.1 (Pin_1); no longer J11.4 (Pin_4)
- net VCC: now also J11.4 (Pin_4); no longer J11.1 (Pin_1)
Changed lines of the file:
@@
 $Descr A4 11693 8268
 encoding utf-8
-Sheet 5 5
+Sheet 2 5
 Title ""
 Date ""
@@
 AR Path="/61D4EE64/61D3FD3C" Ref="U3"  Part="1"
 AR Path="/61D4FC97/61D3FD3C" Ref="U4"  Part="1"
-F 0 "U4" H 5850 3500 50  0001 L BNN
+F 0 "#U1" H 5850 3500 50  0001 L BNN
 F 1 "HX711" H 5850 3500 50  0001 L BNN
 F 2 "" H 5850 3500 50  0001 L BNN
@@
 AR Path="/61D4EE64/61D3FD43" Ref="R5"  Part="1"
 AR Path="/61D4FC97/61D3FD43" Ref="R7"  Part="1"
-F 0 "R7" V 3643 3700 50  0000 C CNN
+F 0 "R1" V 3643 3700 50  0000 C CNN
 F 1 "1k" V 3734 3700 50  0000 C CNN
 F 2 "Resistor_THT:R_Axial_DIN0207_L6.3mm_D2.5mm_P7.62mm_Horizontal" V 3780 3700 50  0001 C CNN
@@
 AR Path="/61D4EE64/61D3FD49" Ref="R6"  Part="1"
 AR Path="/61D4FC97/61D3FD49" Ref="R8"  Part="1"
-F 0 "R8" V 3643 3950 50  0000 C CNN
+F 0 "R2" V 3643 3950 50  0000 C CNN
 F 1 "1k" V 3734 3950 50  0000 C CNN
 F 2 "Resistor_THT:R_Axial_DIN0207_L6.3mm_D2.5mm_P7.62mm_Horizontal" V 3780 3950 50  0001 C CNN
@@
 AR Path="/61D4EE64/61D53FBD" Ref="J15"  Part="1"
 AR Path="/61D4FC97/61D53FBD" Ref="J17"  Part="1"
-F 0 "J17" H 7280 3542 50  0000 L CNN
+F 0 "J11" H 7280 3542 50  0000 L CNN
 F 1 "Conn_01x04" H 7280 3451 50  0000 L CNN
 F 2 "Connector_PinHeader_2.54mm:PinHeader_1x04_P2.54mm_Vertical" H 7200 3550 50  0001 C CNN
@@
 	7000 3500 7000 3550
 Wire Wire Line
-	6550 3500 7000 3500
-Wire Wire Line
 	7000 3650 7000 3700
 Wire Wire Line
@@
 Text GLabel 5850 4500 3    50   Input ~ 0
 GND
-Wire Wire Line
-	7000 3750 7000 4500
-Wire Wire Line
-	7000 4500 5850 4500
-Wire Wire Line
-	5850 2900 7000 2900
-Wire Wire Line
-	7000 2900 7000 3450
 Text Label 4950 3800 0    50   ~ 0
 A-
@@
 AR Path="/61D4E257/61D56664" Ref="J12"  Part="1"
 AR Path="/61D4EE64/61D56664" Ref="J14"  Part="1"
-F 0 "J16" H 4418 4567 50  0000 C CNN
+F 0 "J10" H 4418 4567 50  0000 C CNN
 F 1 "Conn_01x06" H 4418 4476 50  0000 C CNN
 F 2 "Connector_PinHeader_2.54mm:PinHeader_1x06_P2.54mm_Vertical" H 4500 4150 50  0001 C CNN
@@
 	3250 3400 4750 3400
 Wire Wire Line
-	3100 3600 4800 3600
-Wire Wire Line
-	4100 3800 4850 3800
-Wire Wire Line
 	4700 3950 4700 3200
 Connection ~ 4700 3200
@@
 	4750 3400 5150 3400
 Wire Wire Line
-	4800 3600 4800 4150
-Wire Wire Line
 	4800 4150 4700 4150
-Connection ~ 4800 3600
-Wire Wire Line
-	4800 3600 5150 3600
-Wire Wire Line
-	4850 3800 4850 4250
 Wire Wire Line
 	4850 4250 4700 4250
-Connection ~ 4850 3800
-Wire Wire Line
-	4850 3800 5150 3800
 Wire Wire Line
 	4900 4000 4900 4350
@@
 NoConn ~ 5100 4000
 NoConn ~ 5100 4200
+Wire Wire Line
+	3100 3600 4850 3600
+Wire Wire Line
+	4100 3800 4800 3800
+Wire Wire Line
+	4800 4150 4800 3800
+Connection ~ 4800 3800
+Wire Wire Line
+	4800 3800 5150 3800
+Wire Wire Line
+	4850 4250 4850 3600
+Connection ~ 4850 3600
+Wire Wire Line
+	4850 3600 5150 3600
+Wire Wire Line
+	5850 2900 6750 2900
+Wire Wire Line
+	6750 2900 6750 3750
+Wire Wire Line
+	6750 3750 7000 3750
+Wire Wire Line
+	6550 3500 7000 3500
+Wire Wire Line
+	7000 3450 6800 3450
+Wire Wire Line
+	6800 3450 6800 4500
+Wire Wire Line
+	6800 4500 5850 4500
 $EndSCHEMATC

Commit message: JST connectors, increased track width of VCC, moved bluetooth modules, other small fixes
Connections:
- net DT: now also J11.3 (Pin_3); no longer J11.2 (Pin_2)
- net GND: now also J11.4 (Pin_4); no longer J11.1 (Pin_1)
- net SCK: now also J11.2 (Pin_2); no longer J11.3 (Pin_3)
- net VCC: now also J11.1 (Pin_1); no longer J11.4 (Pin_4)
Changed lines of the file:
@@
 Text HLabel 3100 3800 0    50   Input ~ 0
 E+
-Text HLabel 6650 3500 1    50   Input ~ 0
+Text HLabel 6800 3650 3    50   Input ~ 0
 DT
-Text HLabel 6650 3700 3    50   Input ~ 0
+Text HLabel 6650 3550 1    50   Input ~ 0
 SCK
-$Comp
-L Connector_Generic:Conn_01x04 J11
-U 1 1 61D53FBD
-P 7200 3550
-AR Path="/61D3CBFC/61D53FBD" Ref="J11"  Part="1"
-AR Path="/61D4E257/61D53FBD" Ref="J13"  Part="1"
-AR Path="/61D4EE64/61D53FBD" Ref="J15"  Part="1"
-AR Path="/61D4FC97/61D53FBD" Ref="J17"  Part="1"
-F 0 "J11" H 7280 3542 50  0000 L CNN
-F 1 "Conn_01x04" H 7280 3451 50  0000 L CNN
-F 2 "Connector_PinHeader_2.54mm:PinHeader_1x04_P2.54mm_Vertical" H 7200 3550 50  0001 C CNN
-F 3 "~" H 7200 3550 50  0001 C CNN
-	1    7200 3550
-	1    0    0    -1
-$EndComp
-Wire Wire Line
-	7000 3500 7000 3550
-Wire Wire Line
-	7000 3650 7000 3700
-Wire Wire Line
-	6550 3700 7000 3700
 Text GLabel 5850 4500 3    50   Input ~ 0
 GND
@@
 Wire Wire Line
 	5850 2900 6750 2900
+$Comp
+L Connector_Generic:Conn_01x04 J11
+U 1 1 61D53FBD
+P 7200 3550
+AR Path="/61D3CBFC/61D53FBD" Ref="J11"  Part="1"
+AR Path="/61D4E257/61D53FBD" Ref="J13"  Part="1"
+AR Path="/61D4EE64/61D53FBD" Ref="J15"  Part="1"
+AR Path="/61D4FC97/61D53FBD" Ref="J17"  Part="1"
+F 0 "J11" H 7280 3542 50  0000 L CNN
+F 1 "Conn_01x04" H 7280 3451 50  0000 L CNN
+F 2 "Connector_PinHeader_2.54mm:PinHeader_1x04_P2.54mm_Vertical" H 7200 3550 50  0001 C CNN
+F 3 "~" H 7200 3550 50  0001 C CNN
+	1    7200 3550
+	1    0    0    -1
+$EndComp
 Wire Wire Line
-	6750 2900 6750 3750
+	6750 2900 6750 3450
 Wire Wire Line
-	6750 3750 7000 3750
+	6750 3450 7000 3450
 Wire Wire Line
-	6550 3500 7000 3500
+	6550 3500 6550 3650
 Wire Wire Line
-	7000 3450 6800 3450
+	6550 3650 7000 3650
 Wire Wire Line
-	6800 3450 6800 4500
+	6550 3700 6650 3700
 Wire Wire Line
-	6800 4500 5850 4500
+	6650 3700 6650 3550
+Wire Wire Line
+	6650 3550 7000 3550
+Wire Wire Line
+	7000 3750 7000 4500
+Wire Wire Line
+	5850 4500 7000 4500
 $EndSCHEMATC
