File: Load Cell/V2_load_cell.sch (KiCad schematic (older format))
At the start: 18 parts, among them J1 Conn_01x02, J2 Conn_01x06, J3 Conn_01x06, J6 Conn_01x03, J7 Conn_01x03, J8 Conn_01x03, J9 Conn_01x03, SW1 SW_DIP_x01

Commit message: pcb v2 update
Parts:
- J6, J7, J8, J9: footprint Connector_JST:JST_PH_B3B-PH-K_1x03_P2.00mm_Vertical -> Connector_JST:JST_PH_S3B-PH-K_1x03_P2.00mm_Horizontal
Changed lines of the file:
@@
 F 0 "J6" H 2718 1367 50  0000 C CNN
 F 1 "Conn_01x03" H 2718 1276 50  0000 C CNN
-F 2 "Connector_JST:JST_PH_B3B-PH-K_1x03_P2.00mm_Vertical" H 2800 1050 50  0001 C CNN
+F 2 "Connector_JST:JST_PH_S3B-PH-K_1x03_P2.00mm_Horizontal" H 2800 1050 50  0001 C CNN
 F 3 "~" H 2800 1050 50  0001 C CNN
 	1    2800 1050
@@
 F 0 "J7" H 2718 2617 50  0000 C CNN
 F 1 "Conn_01x03" H 2718 2526 50  0000 C CNN
-F 2 "Connector_JST:JST_PH_B3B-PH-K_1x03_P2.00mm_Vertical" H 2800 2300 50  0001 C CNN
+F 2 "Connector_JST:JST_PH_S3B-PH-K_1x03_P2.00mm_Horizontal" H 2800 2300 50  0001 C CNN
 F 3 "~" H 2800 2300 50  0001 C CNN
 	1    2800 2300
@@
 F 0 "J8" H 2718 3867 50  0000 C CNN
 F 1 "Conn_01x03" H 2718 3776 50  0000 C CNN
-F 2 "Connector_JST:JST_PH_B3B-PH-K_1x03_P2.00mm_Vertical" H 2800 3550 50  0001 C CNN
+F 2 "Connector_JST:JST_PH_S3B-PH-K_1x03_P2.00mm_Horizontal" H 2800 3550 50  0001 C CNN
 F 3 "~" H 2800 3550 50  0001 C CNN
 	1    2800 3550
@@
 F 0 "J9" H 2718 5117 50  0000 C CNN
 F 1 "Conn_01x03" H 2718 5026 50  0000 C CNN
-F 2 "Connector_JST:JST_PH_B3B-PH-K_1x03_P2.00mm_Vertical" H 2800 4800 50  0001 C CNN
+F 2 "Connector_JST:JST_PH_S3B-PH-K_1x03_P2.00mm_Horizontal" H 2800 4800 50  0001 C CNN
 F 3 "~" H 2800 4800 50  0001 C CNN
 	1    2800 4800

Commit message: JST connectors, increased track width of VCC, moved bluetooth modules, other small fixes
Parts:
- J6, J7, J8, J9: footprint Connector_JST:JST_PH_S3B-PH-K_1x03_P2.00mm_Horizontal -> Connector_JST:JST_PH_B3B-PH-K_1x03_P2.00mm_Vertical
Connections:
- net DT0: now also A1.6 (D3); no longer A1.5 (D2)
- net DT1: now also A1.8 (D5); no longer A1.7 (D4)
- net DT2: now also A1.10 (D7); no longer A1.9 (D6)
- net DT3: now also A1.12 (D9); no longer A1.11 (D8)
- net GND: now also J2.3 (Pin_3), J3.3 (Pin_3); no longer J2.4 (Pin_4), J3.4 (Pin_4)
- net RX0: now also J2.5 (Pin_5); no longer J2.2 (Pin_2)
- net RX1: now also J3.5 (Pin_5); no longer J3.2 (Pin_2)
- net SCK0: now also A1.5 (D2); no longer A1.6 (D3)
- net SCK1: now also A1.7 (D4); no longer A1.8 (D5)
- net SCK2: now also A1.9 (D6); no longer A1.10 (D7)
- net SCK3: now also A1.11 (D8); no longer A1.12 (D9)
- net TX0: now also J2.4 (Pin_4); no longer J2.3 (Pin_3)
- net TX1: now also J3.4 (Pin_4); no longer J3.3 (Pin_3)
- net VCC: now also J2.2 (Pin_2), J3.2 (Pin_2); no longer J2.5 (Pin_5), J3.5 (Pin_5)
Changed lines of the file:
@@
 F 0 "J6" H 2718 1367 50  0000 C CNN
 F 1 "Conn_01x03" H 2718 1276 50  0000 C CNN
-F 2 "Connector_JST:JST_PH_S3B-PH-K_1x03_P2.00mm_Horizontal" H 2800 1050 50  0001 C CNN
+F 2 "Connector_JST:JST_PH_B3B-PH-K_1x03_P2.00mm_Vertical" H 2800 1050 50  0001 C CNN
 F 3 "~" H 2800 1050 50  0001 C CNN
 	1    2800 1050
@@
 F 0 "J7" H 2718 2617 50  0000 C CNN
 F 1 "Conn_01x03" H 2718 2526 50  0000 C CNN
-F 2 "Connector_JST:JST_PH_S3B-PH-K_1x03_P2.00mm_Horizontal" H 2800 2300 50  0001 C CNN
+F 2 "Connector_JST:JST_PH_B3B-PH-K_1x03_P2.00mm_Vertical" H 2800 2300 50  0001 C CNN
 F 3 "~" H 2800 2300 50  0001 C CNN
 	1    2800 2300
@@
 F 0 "J8" H 2718 3867 50  0000 C CNN
 F 1 "Conn_01x03" H 2718 3776 50  0000 C CNN
-F 2 "Connector_JST:JST_PH_S3B-PH-K_1x03_P2.00mm_Horizontal" H 2800 3550 50  0001 C CNN
+F 2 "Connector_JST:JST_PH_B3B-PH-K_1x03_P2.00mm_Vertical" H 2800 3550 50  0001 C CNN
 F 3 "~" H 2800 3550 50  0001 C CNN
 	1    2800 3550
@@
 F 0 "J9" H 2718 5117 50  0000 C CNN
 F 1 "Conn_01x03" H 2718 5026 50  0000 C CNN
-F 2 "Connector_JST:JST_PH_S3B-PH-K_1x03_P2.00mm_Horizontal" H 2800 4800 50  0001 C CNN
+F 2 "Connector_JST:JST_PH_B3B-PH-K_1x03_P2.00mm_Vertical" H 2800 4800 50  0001 C CNN
 F 3 "~" H 2800 4800 50  0001 C CNN
 	1    2800 4800
@@
 Wire Wire Line
 	3000 1350 3400 1350
+Text Label 7850 3450 2    50   ~ 0
+DT0
 Text Label 7850 3350 2    50   ~ 0
-DT0
-Text Label 7850 3450 2    50   ~ 0
 SCK0
+Text Label 7850 3650 2    50   ~ 0
+DT1
 Text Label 7850 3550 2    50   ~ 0
-DT1
-Text Label 7850 3650 2    50   ~ 0
 SCK1
+Text Label 7850 3850 2    50   ~ 0
+DT2
 Text Label 7850 3750 2    50   ~ 0
-DT2
-Text Label 7850 3850 2    50   ~ 0
 SCK2
+Text Label 7850 4050 2    50   ~ 0
+DT3
 Text Label 7850 3950 2    50   ~ 0
-DT3
-Text Label 7850 4050 2    50   ~ 0
 SCK3
 $Comp
@@
 L Connector_Generic:Conn_01x06 J3
 U 1 1 61D8A932
-P 9450 4800
-F 0 "J3" V 9322 5080 50  0000 L CNN
-F 1 "Conn_01x06" V 9413 5080 50  0000 L CNN
-F 2 "Connector_PinSocket_2.54mm:PinSocket_1x06_P2.54mm_Horizontal" H 9450 4800 50  0001 C CNN
-F 3 "~" H 9450 4800 50  0001 C CNN
-	1    9450 4800
-	-1   0    0    -1
+P 9450 4900
+F 0 "J3" V 9322 5180 50  0000 L CNN
+F 1 "Conn_01x06" V 9413 5180 50  0000 L CNN
+F 2 "Connector_PinSocket_2.54mm:PinSocket_1x06_P2.54mm_Horizontal" H 9450 4900 50  0001 C CNN
+F 3 "~" H 9450 4900 50  0001 C CNN
+	1    9450 4900
+	-1   0    0    1
 $EndComp
 $Comp
@@
 GND
 $Comp
-L Connector_Generic:Conn_01x06 J2
-U 1 1 61D79983
-P 9450 2950
-F 0 "J2" V 9322 2562 50  0000 R CNN
-F 1 "Conn_01x06" V 9413 2562 50  0000 R CNN
-F 2 "Connector_PinSocket_2.54mm:PinSocket_1x06_P2.54mm_Horizontal" H 9450 2950 50  0001 C CNN
-F 3 "~" H 9450 2950 50  0001 C CNN
-	1    9450 2950
-	-1   0    0    -1
-$EndComp
-$Comp
 L HC-05:HC-05 #U5
 U 1 1 61D78035
@@
 GND
 Wire Wire Line
-	9650 2850 9850 2850
-Wire Wire Line
-	9650 2950 9750 2950
-Wire Wire Line
 	9650 3050 10100 3050
 Wire Wire Line
@@
 Wire Wire Line
 	9100 3400 9750 3400
-Wire Wire Line
-	9750 3400 9750 2950
-Connection ~ 9750 2950
-Wire Wire Line
-	9750 2950 10100 2950
-Wire Wire Line
-	9850 2850 9850 3550
-Connection ~ 9850 2850
-Wire Wire Line
-	9850 2850 10100 2850
 Wire Wire Line
 	9650 4800 9900 4800
@@
 Text Label 8250 2850 0    50   ~ 0
 VIN
+Wire Wire Line
+	9850 2850 10100 2850
+Wire Wire Line
+	9650 2850 9850 2850
+Connection ~ 9850 2850
+Wire Wire Line
+	9850 2850 9850 3550
+Wire Wire Line
+	9750 2950 10100 2950
+Wire Wire Line
+	9650 2950 9750 2950
+Connection ~ 9750 2950
+Wire Wire Line
+	9750 3400 9750 2950
+$Comp
+L Connector_Generic:Conn_01x06 J2
+U 1 1 61D79983
+P 9450 3050
+F 0 "J2" V 9322 2662 50  0000 R CNN
+F 1 "Conn_01x06" V 9413 2662 50  0000 R CNN
+F 2 "Connector_PinSocket_2.54mm:PinSocket_1x06_P2.54mm_Horizontal" H 9450 3050 50  0001 C CNN
+F 3 "~" H 9450 3050 50  0001 C CNN
+	1    9450 3050
+	-1   0    0    1
+$EndComp
 $EndSCHEMATC

Commit message: v2
Connections:
- net A+0: now also J6.3 (Pin_3); no longer J6.1 (Pin_1)
- net A+1: now also J7.3 (Pin_3); no longer J7.1 (Pin_1)
- net A+2: now also J8.3 (Pin_3); no longer J8.1 (Pin_1)
- net A+3: now also J9.3 (Pin_3); no longer J9.1 (Pin_1)
- net A1: now also A1.8 (D5); no longer A1.20 (A1)
- net A3: now also A1.6 (D3); no longer A1.22 (A3)
- net DT0: now also A1.10 (D7); no longer A1.6 (D3)
- net DT1: now also A1.20 (A1); no longer A1.8 (D5)
- net DT2: now also A1.22 (A3); no longer A1.10 (D7)
- net DT3: now also A1.24 (SCL/A5); no longer A1.12 (D9)
- net E+0: now also J6.1 (Pin_1); no longer J6.3 (Pin_3)
- net E+1: now also J7.1 (Pin_1); no longer J7.3 (Pin_3)
- net E+2: now also J8.1 (Pin_1); no longer J8.3 (Pin_3)
- net E+3: now also J9.1 (Pin_1); no longer J9.3 (Pin_3)
- net SCK0: now also A1.11 (D8); no longer A1.5 (D2)
- net SCK1: now also A1.19 (A0); no longer A1.7 (D4)
- net SCK2: now also A1.21 (A2); no longer A1.9 (D6)
- net SCK3: now also A1.23 (SDA/A4); no longer A1.11 (D8)
- net ST: now also A1.5 (D2); no longer A1.23 (SDA/A4)
- net TX0: now also A1.7 (D4); no longer A1.19 (A0)
- net TX1: now also A1.9 (D6); no longer A1.21 (A2)
- no-connect marks 16 -> 15
Other:
- moved on the sheet: A1, D1, H1, H2, H3, H4, J2, J3, R10, R11, R12, R9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

Commit message: changed some labels, redid traces, flipped JST, new zip
Connections:
- net RX0: now also A1.7 (D4), R9.2; no longer J2.5 (Pin_5), R11.1, R9.1
- net RX1: now also A1.9 (D6), R10.2; no longer J3.5 (Pin_5), R10.1, R12.2
- net TX0: now also A1.6 (D3); no longer A1.7 (D4)
- net TX1: now also A1.8 (D5); no longer A1.9 (D6)
- removed net A1: A1.8 (D5), R9.2
- removed net A3: A1.6 (D3), R10.2
- new net RX0R: J2.5 (Pin_5), R11.1, R9.1
- new net RX1R: J3.5 (Pin_5), R10.1, R12.2
Changed lines of the file:
@@
 	8650 4100 8550 4100
 Text Label 8550 3900 2    50   ~ 0
-A1
+RX0
 Text Label 8550 4100 2    50   ~ 0
-A3
+RX1
 Text Label 9000 4100 0    50   ~ 0
-RX1
+RX1R
 Text Label 8550 4000 2    50   ~ 0
 TX1
@@
 $EndComp
 Text Label 9150 3900 0    50   ~ 0
-RX0
+RX0R
 Text Label 8550 3800 2    50   ~ 0
 TX0
@@
 Text Label 5350 3800 2    50   ~ 0
 DT0
-Text Label 5350 3600 2    50   ~ 0
-A1
-Text Label 5350 3400 2    50   ~ 0
-A3
+Text Label 5350 3500 2    50   ~ 0
+RX0
+Text Label 5350 3700 2    50   ~ 0
+RX1
 Text Label 5350 3300 2    50   ~ 0
 ST
-Text Label 5350 3500 2    50   ~ 0
+Text Label 5350 3400 2    50   ~ 0
 TX0
 NoConn ~ 5350 4000
@@
 Text Label 3000 2400 0    50   ~ 0
 E+1
-Text Label 5350 3700 2    50   ~ 0
+Text Label 5350 3600 2    50   ~ 0
 TX1
 $EndSCHEMATC
